File: output/pcbs/bottom_plate.kicad_pcb (KiCad board)
At the start: 2 copper layers, 379.3 x 126.2 mm, 11 parts

Commit message: second commit
Parts:
- moved _11 19.0 mm to (205.8, 172.3)
- moved _1 4.20 mm to (52.7, 70.9)
- moved _6 3.61 mm to (358.9, 70.9)
- moved _7 0.91 mm to (363.6, 128.0)
- moved _10 0.73 mm to (290.6, 159.9)
- moved _8 0.68 mm to (285.1, 79.6)
- moved _9 0.68 mm to (244.2, 78.3)
- moved _4 0.24 mm to (167.5, 78.3)
- moved _3 0.24 mm to (126.6, 79.6)
- moved _5 0.23 mm to (121.1, 159.9)
Other:
- board size 379.3 x 126.2 mm -> 375.4 x 121.4 mm

Commit message: .
Parts:
- added _12: , MountingHole_2.2mm_M2_Pad_Via, F.Cu at (192.8, 238.5)
- added _13: , MountingHole_2.2mm_M2_Pad_Via, F.Cu at (138.7, 255.9)
- moved _6 321.5 mm to (84.6, 238.5), turned to -75 degrees
- moved _10 164.9 mm to (126.9, 141.1), turned to 45 degrees
- moved _7 146.5 mm to (217.1, 129.0), turned to 45 degrees
- moved _9 127.4 mm to (153.8, 168.0), turned to 45 degrees
- moved _8 106.9 mm to (245.4, 178.8), turned to 45 degrees
- moved _3 88.5 mm to (123.6, 168.0), turned to -45 degrees
- moved _11 71.9 mm to (153.8, 221.9), turned to 45 degrees
- moved _4 65.1 mm to (150.5, 141.1), turned to -45 degrees
- moved _5 62.1 mm to (123.6, 221.9), turned to -45 degrees
- moved _1 58.6 mm to (60.3, 129.0), turned to -45 degrees
- moved _2 53.3 mm to (32.0, 178.8), turned to -45 degrees
Other:
- board size 375.4 x 121.4 mm -> 264 x 153.8 mm
