File: output/pcbs/pcb_plate.kicad_pcb (KiCad board)
At the start: 2 copper layers, 379.3 x 126.2 mm, 75 parts

Commit message: second commit
Parts:
- added D37: , ComboDiode, F.Cu at (247.0, 161.0)
- added D38: , ComboDiode, F.Cu at (220.0, 173.9)
- added S37: , MX, F.Cu at (243.8, 157.2)
- added S38: , MX, F.Cu at (219.1, 168.9)
- moved D19 196.0 mm to (191.7, 173.9), turned to -10 degrees
- moved S19 193.5 mm to (192.6, 168.9), turned to -10 degrees
- moved D36 67.6 mm to (308.6, 169.9), turned to 50 degrees
- moved S36 67.1 mm to (304.7, 166.7), turned to 50 degrees
- moved D34 61.3 mm to (293.3, 102.1), turned to 20 degrees
- moved S34 61.3 mm to (291.6, 97.4), turned to 20 degrees
- moved D28 47.8 mm to (325.8, 80.1)
- moved S28 47.8 mm to (324.1, 75.4)
- moved D31 46.1 mm to (309.9, 92.0)
- moved S31 46.1 mm to (308.2, 87.3)
- moved D25 36.1 mm to (346.3, 80.8)
- moved S25 36.1 mm to (344.6, 76.1)
- moved D22 31.5 mm to (368.8, 86.8)
- moved S22 31.5 mm to (367.1, 82.1)
- moved S35 23.1 mm to (321.4, 151.5), turned to 35 degrees
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Connections:
- D19 pad 1: P8 -> P10
- D19 pad 2: mirror_pinky_bottom -> two_one
- D20 pad 1: P7 -> P8
- D20 pad 2: mirror_pinky_home -> mirror_pinky_bottom
- D21 pad 1: P6 -> P7
- D21 pad 2: mirror_pinky_top -> mirror_pinky_home
- D22 pad 1: P8 -> P6
- D22 pad 2: mirror_ring_bottom -> mirror_pinky_top
- D23 pad 1: P7 -> P8
- D23 pad 2: mirror_ring_home -> mirror_ring_bottom
- D24 pad 1: P6 -> P7
- D24 pad 2: mirror_ring_top -> mirror_ring_home
- D25 pad 1: P8 -> P6
- D25 pad 2: mirror_middle_bottom -> mirror_ring_top
- D26 pad 1: P7 -> P8
- D26 pad 2: mirror_middle_home -> mirror_middle_bottom
- D27 pad 1: P6 -> P7
- D27 pad 2: mirror_middle_top -> mirror_middle_home
- D28 pad 1: P8 -> P6
- D28 pad 2: mirror_index_bottom -> mirror_middle_top
- D29 pad 1: P7 -> P8
- D29 pad 2: mirror_index_home -> mirror_index_bottom
- D30 pad 1: P6 -> P7
- D30 pad 2: mirror_index_top -> mirror_index_home
- D31 pad 1: P8 -> P6
- D31 pad 2: mirror_inner_bottom -> mirror_index_top
- D32 pad 1: P7 -> P8
- D32 pad 2: mirror_inner_home -> mirror_inner_bottom
- D33 pad 1: P6 -> P7
- D33 pad 2: mirror_inner_top -> mirror_inner_home
- D34 pad 1: P9 -> P6
- D34 pad 2: mirror_layer_cluster -> mirror_inner_top
- D35 pad 2: mirror_space_cluster -> mirror_layer_cluster
- D36 pad 2: mirror_one_one -> mirror_space_cluster
- S16 pad 1: P18 -> P5
- S17 pad 1: P19 -> P18
- S18 pad 1: P20 -> P19
- S19 pad 1: P4 -> P20
- S19 pad 2: mirror_pinky_bottom -> two_one
- S20 pad 2: mirror_pinky_home -> mirror_pinky_bottom
- S21 pad 2: mirror_pinky_top -> mirror_pinky_home
- S22 pad 1: P5 -> P4
- S22 pad 2: mirror_ring_bottom -> mirror_pinky_top
- S23 pad 2: mirror_ring_home -> mirror_ring_bottom
- S24 pad 2: mirror_ring_top -> mirror_ring_home
- S25 pad 1: P18 -> P5
- S25 pad 2: mirror_middle_bottom -> mirror_ring_top
- S26 pad 2: mirror_middle_home -> mirror_middle_bottom
- S27 pad 2: mirror_middle_top -> mirror_middle_home
- S28 pad 1: P19 -> P18
- S28 pad 2: mirror_index_bottom -> mirror_middle_top
- S29 pad 2: mirror_index_home -> mirror_index_bottom
- S30 pad 2: mirror_index_top -> mirror_index_home
- S31 pad 1: P20 -> P19
- S31 pad 2: mirror_inner_bottom -> mirror_index_top
- S32 pad 2: mirror_inner_home -> mirror_inner_bottom
- S33 pad 2: mirror_inner_top -> mirror_inner_home
- S34 pad 1: P18 -> P20
- S34 pad 2: mirror_layer_cluster -> mirror_inner_top
- S35 pad 1: P19 -> P5
- S35 pad 2: mirror_space_cluster -> mirror_layer_cluster
- S36 pad 1: P20 -> P18
- S36 pad 2: mirror_one_one -> mirror_space_cluster
Other:
- board size 379.3 x 126.2 mm -> 375.4 x 121.4 mm

Commit message: end
Parts:
- moved D34 18.0 mm to (299.7, 119.0)
- moved S25 18.0 mm to (351.0, 93.0)
- moved D18 18.0 mm to (171.1, 177.9)
- moved D7 18.0 mm to (79.2, 132.8)
- moved D9 18.0 mm to (92.2, 97.0)
- moved D15 18.0 mm to (124.8, 119.0)
- moved S29 18.0 mm to (327.6, 140.0)
- moved D10 18.0 mm to (95.2, 144.7)
- moved S1 18.0 mm to (38.0, 134.8)
- moved D20 18.0 mm to (388.2, 139.5)
- moved D16 18.0 mm to (93.8, 172.4)
- moved D14 18.0 mm to (118.3, 136.9)
- moved S16 18.0 mm to (96.7, 168.3)
- moved D6 18.0 mm to (71.7, 97.7)
- moved S32 18.0 mm to (311.0, 150.1)
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Routing:
- net P18: track 0.00 -> 496.7 mm, vias 0 -> 4
- net P5: track 0.00 -> 481.6 mm, vias 0 -> 3
- net P19: track 0.00 -> 427.9 mm, vias 0 -> 2
- net P4: track 0.00 -> 427.3 mm
- net P20: track 0.00 -> 380.2 mm
- net P16: track 0.00 -> 222.9 mm
- net P9: track 0.00 -> 222.2 mm, vias 0 -> 1
- net P10: track 0.00 -> 218.7 mm
- net P8: track 0.00 -> 216.8 mm
- net P14: track 0.00 -> 210.0 mm
- net P7: track 0.00 -> 204.0 mm
- net P15: track 0.00 -> 197.2 mm
- net P6: track 0.00 -> 191.1 mm
- net GND: track 0.00 -> 59.0 mm
- net P2: track 0.00 -> 33.1 mm, vias 0 -> 1
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Other:
- net class Default removed

Commit message: .
Parts:
- removed D37, D38: , ComboDiode
- removed S37, S38: , MX
- moved S28 160.4 mm to (205.0, 192.3), turned to 45 degrees
- moved S25 159.2 mm to (214.4, 174.8), turned to 45 degrees
- moved S31 159.2 mm to (194.2, 208.4), turned to 45 degrees
- moved D28 157.9 mm to (211.3, 198.6), turned to 45 degrees
- moved D31 156.8 mm to (200.6, 214.8), turned to 45 degrees
- moved D25 156.1 mm to (220.8, 181.1), turned to 45 degrees
- moved S22 155.7 mm to (233.3, 166.7), turned to 45 degrees
- moved S27 154.2 mm to (187.5, 147.8), turned to 45 degrees
- moved S24 153.9 mm to (206.3, 139.7), turned to 45 degrees
- moved D22 152.2 mm to (239.6, 173.0), turned to 45 degrees
- moved S21 151.9 mm to (229.2, 135.7), turned to 45 degrees
- moved D27 150.1 mm to (193.8, 154.2), turned to 45 degrees
- moved D24 149.7 mm to (212.7, 146.1), turned to 45 degrees
- moved S30 149.4 mm to (178.0, 165.3), turned to 45 degrees
- moved D21 147.5 mm to (235.6, 142.1), turned to 45 degrees
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Connections:
- D19 pad 1: P10 -> P8
- D19 pad 2: two_one -> mirror_pinky_bottom
- D20 pad 1: P8 -> P7
- D20 pad 2: mirror_pinky_bottom -> mirror_pinky_home
- D21 pad 1: P7 -> P6
- D21 pad 2: mirror_pinky_home -> mirror_pinky_top
- D22 pad 1: P6 -> P8
- D22 pad 2: mirror_pinky_top -> mirror_ring_bottom
- D23 pad 1: P8 -> P7
- D23 pad 2: mirror_ring_bottom -> mirror_ring_home
- D24 pad 1: P7 -> P6
- D24 pad 2: mirror_ring_home -> mirror_ring_top
- D25 pad 1: P6 -> P8
- D25 pad 2: mirror_ring_top -> mirror_middle_bottom
- D26 pad 1: P8 -> P7
- D26 pad 2: mirror_middle_bottom -> mirror_middle_home
- D27 pad 1: P7 -> P6
- D27 pad 2: mirror_middle_home -> mirror_middle_top
- D28 pad 1: P6 -> P8
- D28 pad 2: mirror_middle_top -> mirror_index_bottom
- D29 pad 1: P8 -> P7
- D29 pad 2: mirror_index_bottom -> mirror_index_home
- D30 pad 1: P7 -> P6
- D30 pad 2: mirror_index_home -> mirror_index_top
- D31 pad 1: P6 -> P8
- D31 pad 2: mirror_index_top -> mirror_inner_bottom
- D32 pad 1: P8 -> P7
- D32 pad 2: mirror_inner_bottom -> mirror_inner_home
- D33 pad 1: P7 -> P6
- D33 pad 2: mirror_inner_home -> mirror_inner_top
- D34 pad 1: P6 -> P9
- D34 pad 2: mirror_inner_top -> mirror_layer_cluster
- D35 pad 2: mirror_layer_cluster -> mirror_space_cluster
- D36 pad 2: mirror_space_cluster -> mirror_one_one
- S19 pad 1: P20 -> P4
- S19 pad 2: two_one -> mirror_pinky_bottom
- S20 pad 2: mirror_pinky_bottom -> mirror_pinky_home
- S21 pad 2: mirror_pinky_home -> mirror_pinky_top
- S22 pad 1: P4 -> P5
- S22 pad 2: mirror_pinky_top -> mirror_ring_bottom
- S23 pad 2: mirror_ring_bottom -> mirror_ring_home
- S24 pad 2: mirror_ring_home -> mirror_ring_top
- S25 pad 1: P5 -> P18
- S25 pad 2: mirror_ring_top -> mirror_middle_bottom
- S26 pad 2: mirror_middle_bottom -> mirror_middle_home
- S27 pad 2: mirror_middle_home -> mirror_middle_top
- S28 pad 1: P18 -> P19
- S28 pad 2: mirror_middle_top -> mirror_index_bottom
- S29 pad 2: mirror_index_bottom -> mirror_index_home
- S30 pad 2: mirror_index_home -> mirror_index_top
- S31 pad 1: P19 -> P20
- S31 pad 2: mirror_index_top -> mirror_inner_bottom
- S32 pad 2: mirror_inner_bottom -> mirror_inner_home
- S33 pad 2: mirror_inner_home -> mirror_inner_top
- S34 pad 1: P20 -> P5
- S34 pad 2: mirror_inner_top -> mirror_layer_cluster
- S35 pad 1: P5 -> P18
- S35 pad 2: mirror_layer_cluster -> mirror_space_cluster
- S36 pad 1: P18 -> P19
- S36 pad 2: mirror_space_cluster -> mirror_one_one
Routing:
- net P18: track 496.7 -> 0.00 mm, vias 4 -> 0
- net P5: track 481.6 -> 0.00 mm, vias 3 -> 0
- net P19: track 427.9 -> 0.00 mm, vias 2 -> 0
- net P4: track 427.3 -> 0.00 mm
- net P20: track 380.2 -> 0.00 mm
- net P16: track 222.9 -> 0.00 mm
- net P9: track 222.2 -> 0.00 mm, vias 1 -> 0
- net P10: track 218.7 -> 0.00 mm
- net P8: track 216.8 -> 0.00 mm
- net P14: track 210.0 -> 0.00 mm
- net P7: track 204.0 -> 0.00 mm
- net P15: track 197.2 -> 0.00 mm
- net P6: track 191.1 -> 0.00 mm
- net GND: track 59.0 -> 0.00 mm
- net P2: track 33.1 -> 0.00 mm, vias 1 -> 0
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Other:
- board size 375.4 x 121.4 mm -> 264 x 153.8 mm
- net class Default added: clearance 0.2, trace_width 0.25, via_dia 0.8, via_drill 0.4
