File: output/pcbs/top_plate.kicad_pcb (KiCad board)
At the start: 2 copper layers, 379.3 x 126.2 mm, 17 parts

Commit message: second commit
Parts:
- moved _17 19.0 mm to (205.8, 172.3)
- moved _5 4.20 mm to (52.7, 70.9)
- moved _11 3.61 mm to (358.9, 70.9)
- moved _12 0.91 mm to (363.6, 128.0)
- moved _16 0.73 mm to (290.6, 159.9)
- moved _15 0.70 mm to (262.4, 128.3)
- moved _13 0.68 mm to (285.1, 79.6)
- moved _14 0.68 mm to (244.2, 78.3)
- moved _1 0.46 mm to (227.9, 93.3)
- moved _2 0.46 mm to (183.8, 93.3)
- moved _3 0.46 mm to (227.9, 137.4)
- moved _4 0.46 mm to (183.8, 137.4)
- moved _8 0.24 mm to (167.5, 78.3)
- moved _7 0.24 mm to (126.6, 79.6)
- moved _10 0.23 mm to (121.1, 159.9)
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Other:
- board size 379.3 x 126.2 mm -> 375.4 x 121.4 mm

Commit message: .
Parts:
- removed _14, _15, _16, _17: , MountingHole_2.2mm_M2_Pad_Via
- moved _11 254.7 mm to (153.8, 221.9), turned to 45 degrees
- moved _13 219.9 mm to (153.7, 255.9), turned to 0 degrees
- moved _12 203.4 mm to (192.8, 238.5), turned to 75 degrees
- moved _2 174.2 mm to (32.0, 178.8), turned to -45 degrees
- moved _1 171.4 mm to (60.3, 129.0), turned to -45 degrees
- moved _5 166.8 mm to (123.6, 221.9), turned to -45 degrees
- moved _8 127.1 mm to (245.4, 178.8), turned to 45 degrees
- moved _6 116.4 mm to (84.6, 238.5), turned to -75 degrees
- moved _3 108.7 mm to (123.6, 168.0), turned to -45 degrees
- moved _7 103.1 mm to (217.1, 129.0), turned to 45 degrees
- moved _9 39.9 mm to (153.8, 168.0), turned to 45 degrees
- moved _4 33.5 mm to (150.5, 141.1), turned to -45 degrees
- moved _10 19.7 mm to (126.9, 141.1), turned to 45 degrees
Other:
- board size 375.4 x 121.4 mm -> 264 x 153.8 mm
